File: 2-Hardware/BusPirateConnectors.sch (KiCad schematic (older format))
At the start: 8 parts

Commit message: Annotations and pull-up changes
Added some text notes to the schematic.
Removed 3v3/5v select jumper from VPU
Parts:
- removed JP? (x3): JUMPER3, symbol JUMPER3
Connections:
- net MEM_SPI_VPU is gone; now on net +3.3V: P?.5 (P5)
- net SD_SPI_VPU is gone; now on net +3.3V: P?.5 (P5)
- net SYS_I2C_VPU is gone; now on net +3.3V: P?.5 (P5)
Other:
- note added: "+3.3V and +5v are from the Bus Pirate power supply. \nTo avoid bus contention, do not enable in SW unless required.\n"
- note added: "Default pullup is 3v3. Bus Pirate v4 supports 3v3 \nor 5v from SW, in addition to default external input."
- note added: "Headers for flying \nwires to select chip."
Changed lines of the file:
@@
 	2350 3000 2350 3150
-$Comp
-L JUMPER3 JP?
-U 1 1 5436C1A6
-P 2350 2900
-F 0 "JP?" H 2400 2800 40  0000 L CNN
-F 1 "JUMPER3" H 2350 3000 40  0000 C CNN
-F 2 "" H 2350 2900 60  0000 C CNN
-F 3 "" H 2350 2900 60  0000 C CNN
-	1    2350 2900
-	1    0    0    -1
-$EndComp
-Wire Wire Line
-	2100 2900 2000 2900
-Wire Wire Line
-	2000 2900 2000 2850
-Wire Wire Line
-	2600 2900 2700 2900
-Wire Wire Line
-	2700 2900 2700 2850
 $Comp
 L +3.3V #PWR08
 U 1 1 5436C24B
-P 2700 2850
-F 0 "#PWR08" H 2700 2810 30  0001 C CNN
-F 1 "+3.3V" H 2700 2960 30  0000 C CNN
-F 2 "" H 2700 2850 60  0000 C CNN
-F 3 "" H 2700 2850 60  0000 C CNN
-	1    2700 2850
-	1    0    0    -1
-$EndComp
-$Comp
-L +5V #PWR09
-U 1 1 5436C25A
-P 2000 2850
-F 0 "#PWR09" H 2000 2940 20  0001 C CNN
-F 1 "+5V" H 2000 2940 30  0000 C CNN
-F 2 "" H 2000 2850 60  0000 C CNN
-F 3 "" H 2000 2850 60  0000 C CNN
-	1    2000 2850
+P 2350 3000
+F 0 "#PWR08" H 2350 2960 30  0001 C CNN
+F 1 "+3.3V" H 2350 3110 30  0000 C CNN
+F 2 "" H 2350 3000 60  0000 C CNN
+F 3 "" H 2350 3000 60  0000 C CNN
+	1    2350 3000
 	1    0    0    -1
 $EndComp
@@
 	2350 4900 2350 5050
 $Comp
-L JUMPER3 JP?
-U 1 1 5436C80A
-P 2350 4800
-F 0 "JP?" H 2400 4700 40  0000 L CNN
-F 1 "JUMPER3" H 2350 4900 40  0000 C CNN
-F 2 "" H 2350 4800 60  0000 C CNN
-F 3 "" H 2350 4800 60  0000 C CNN
-	1    2350 4800
-	1    0    0    -1
-$EndComp
-Wire Wire Line
-	2100 4800 2000 4800
-Wire Wire Line
-	2000 4800 2000 4750
-Wire Wire Line
-	2600 4800 2700 4800
-Wire Wire Line
-	2700 4800 2700 4750
-$Comp
 L +3.3V #PWR013
 U 1 1 5436C814
-P 2700 4750
-F 0 "#PWR013" H 2700 4710 30  0001 C CNN
-F 1 "+3.3V" H 2700 4860 30  0000 C CNN
-F 2 "" H 2700 4750 60  0000 C CNN
-F 3 "" H 2700 4750 60  0000 C CNN
-	1    2700 4750
-	1    0    0    -1
-$EndComp
-$Comp
-L +5V #PWR014
-U 1 1 5436C81A
-P 2000 4750
-F 0 "#PWR014" H 2000 4840 20  0001 C CNN
-F 1 "+5V" H 2000 4840 30  0000 C CNN
-F 2 "" H 2000 4750 60  0000 C CNN
-F 3 "" H 2000 4750 60  0000 C CNN
-	1    2000 4750
+P 2350 4900
+F 0 "#PWR013" H 2350 4860 30  0001 C CNN
+F 1 "+3.3V" H 2350 5010 30  0000 C CNN
+F 2 "" H 2350 4900 60  0000 C CNN
+F 3 "" H 2350 4900 60  0000 C CNN
+	1    2350 4900
 	1    0    0    -1
 $EndComp
@@
 	7250 3050 7250 3200
 $Comp
-L JUMPER3 JP?
-U 1 1 5436CB7D
-P 7250 2950
-F 0 "JP?" H 7300 2850 40  0000 L CNN
-F 1 "JUMPER3" H 7250 3050 40  0000 C CNN
-F 2 "" H 7250 2950 60  0000 C CNN
-F 3 "" H 7250 2950 60  0000 C CNN
-	1    7250 2950
-	1    0    0    -1
-$EndComp
-Wire Wire Line
-	7000 2950 6900 2950
-Wire Wire Line
-	6900 2950 6900 2900
-Wire Wire Line
-	7500 2950 7600 2950
-Wire Wire Line
-	7600 2950 7600 2900
-$Comp
 L +3.3V #PWR018
 U 1 1 5436CB87
-P 7600 2900
-F 0 "#PWR018" H 7600 2860 30  0001 C CNN
-F 1 "+3.3V" H 7600 3010 30  0000 C CNN
-F 2 "" H 7600 2900 60  0000 C CNN
-F 3 "" H 7600 2900 60  0000 C CNN
-	1    7600 2900
-	1    0    0    -1
-$EndComp
-$Comp
-L +5V #PWR019
-U 1 1 5436CB8D
-P 6900 2900
-F 0 "#PWR019" H 6900 2990 20  0001 C CNN
-F 1 "+5V" H 6900 2990 30  0000 C CNN
-F 2 "" H 6900 2900 60  0000 C CNN
-F 3 "" H 6900 2900 60  0000 C CNN
-	1    6900 2900
+P 7250 3050
+F 0 "#PWR018" H 7250 3010 30  0001 C CNN
+F 1 "+3.3V" H 7250 3160 30  0000 C CNN
+F 2 "" H 7250 3050 60  0000 C CNN
+F 3 "" H 7250 3050 60  0000 C CNN
+	1    7250 3050
 	1    0    0    -1
 $EndComp
@@
 Wire Notes Line
 	1850 4200 5450 4200
+Text Notes 2050 2650 0    39   ~ 0
++3.3V and +5v are from the Bus Pirate power supply. \nTo avoid bus contention, do not enable in SW unless required.\n
+Text Notes 3300 6050 0    39   ~ 0
+Headers for flying \nwires to select chip.
+Text Notes 1900 4650 0    39   ~ 0
+Default pullup is 3v3. Bus Pirate v4 supports 3v3 \nor 5v from SW, in addition to default external input.
 $EndSCHEMATC
